Commit message: hls lidar update

File: description/urdf/rover.urdf (robot description, URDF)
Before this commit: robot rover_prototype, 6 links, 5 joints
Links:
- added link scan_link; visual cylinder length=0.04 radius=0.03
- link base_link: geometry visual box size=0.28 0.28 0.12
Joints:
- added joint lidar_to_base: type fixed, parent base_link, child scan_link, origin xyz=0.06 0 0.12 rpy=0 0 0

Commit message: Added tf from imu to baselink

File: description/urdf/rover.urdf (robot description, URDF)
Before this commit: robot rover_prototype, 7 links, 6 joints
Links:
- added link imu; visual cylinder length=0.01 radius=0.01
Joints:
- added joint imu_to_base_link: type fixed, parent imu, child base_link, origin xyz=0 0 0 rpy=0 0 0

Commit message: lidar flip

File: description/urdf/rover.urdf (robot description, URDF)
Before this commit: robot rover_prototype, 8 links, 7 joints
Joints:
- joint imu_to_base_link: child base_link -> imu; origin xyz=0 0 0 rpy=0 0 0 -> xyz=0 0 0.01 rpy=0 0 0; parent imu -> base_link
- joint lidar_to_base: origin xyz=0.06 0 0.12 rpy=0 0 0 -> xyz=-0.06 0 0.12 rpy=0 0 0
- joint lwheel_to_base: origin xyz=0 0.14 0 rpy=1.57 0 0 -> xyz=0 0.14 0.02 rpy=1.57 0 0
- joint rwheel_to_base: origin xyz=0 -0.14 0 rpy=-1.57 0 0 -> xyz=0 -0.14 0.02 rpy=-1.57 0 0

Commit message: base link collision

File: description/urdf/rover.urdf (robot description, URDF)
Before this commit: robot rover_prototype, 8 links, 7 joints
Links:
- link base_link: geometry collision box size=0.32 0.32 0.12; visual box size=0.28 0.28 0.12

Commit message: Add camera + lidar launch file into perception.launch, start camera depth cloud + lidar fusion

File: description/urdf/rover.urdf (robot description, URDF)
Before this commit: robot rover_prototype, 8 links, 7 joints
Links:
- link base_link: geometry collision cylinder length=0.6 radius=0.2; visual box size=0.28 0.28 0.12
